File: coracao_8bits.sch (EAGLE design)
At the start: 70 parts, among them IC1 74HC595D, IC2 74HC595D, IC3 74HC595D, IC4 74HC595D, J1 FEMALE 2x3, U2 ATMEGA168, Y1 16MHZ

Commit message: add power jack
Parts:
- added DISP1: YSD-439AR6B-35, SparkFun-LED:7-SEGMENT-4DIGIT-10MM-RED
- added J2: POWER_JACK, SparkFun-Connectors:POWER_JACK
- added LOGO1: OSHW-LOGOMINI, SparkFun-Aesthetics:OSHW-LOGOMINI
Connections:
- removed net VIN: C1.+, U1.EN, U1.IN
- new net DEETE: C1.+, J2.PWR, U1.EN, U1.IN
- net GND: now also J2.GND, J2.GNDBREAK
Other:
- note added: "Clock"
Changed lines of the file:
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@@
 <part name="SUPPLY3" library="SparkFun-Aesthetics" deviceset="VCC" device=""/>
 <part name="S2" library="SparkFun-Switches" deviceset="MOMENTARY-SWITCH-SPST" device="-SMD-6.0X3.5MM" value="Reset"/>
+<part name="LOGO1" library="SparkFun-Aesthetics" deviceset="OSHW-LOGO" device="MINI"/>
+<part name="FRAME5" library="SparkFun-Aesthetics" deviceset="FRAME-A4L" device=""/>
+<part name="DISP1" library="SparkFun-LED" deviceset="7-SEGMENT-4DIGIT-10MM" device="-RED" value="YSD-439AR6B-35"/>
+<part name="J2" library="SparkFun-Connectors" deviceset="POWER_JACK" device=""/>
+<part name="GND39" library="SparkFun-Aesthetics" deviceset="GND" device=""/>
 </parts>
 <sheets>
@@
 <instance part="C3" gate="G$1" x="180.34" y="116.84"/>
 <instance part="GND5" gate="1" x="180.34" y="104.14"/>
+<instance part="LOGO1" gate="G$1" x="259.08" y="33.02"/>
+<instance part="J2" gate="G$1" x="86.36" y="124.46"/>
+<instance part="GND39" gate="1" x="93.98" y="104.14"/>
 </instances>
 <busses>
 </busses>
 <nets>
-<net name="VIN" class="0">
-<segment>
-<pinref part="U1" gate="G$1" pin="IN"/>
-<wire x1="129.54" y1="132.08" x2="121.92" y2="132.08" width="0.1524" layer="91"/>
-<label x="99.06" y="132.08" size="1.9304" layer="95" rot="R180" xref="yes"/>
-<pinref part="U1" gate="G$1" pin="EN"/>
-<wire x1="121.92" y1="132.08" x2="109.22" y2="132.08" width="0.1524" layer="91"/>
-<wire x1="109.22" y1="132.08" x2="99.06" y2="132.08" width="0.1524" layer="91"/>
-<wire x1="129.54" y1="127" x2="121.92" y2="127" width="0.1524" layer="91"/>
-<wire x1="121.92" y1="127" x2="121.92" y2="132.08" width="0.1524" layer="91"/>
-<junction x="121.92" y="132.08"/>
-<pinref part="C1" gate="G$1" pin="+"/>
-<wire x1="109.22" y1="121.92" x2="109.22" y2="132.08" width="0.1524" layer="91"/>
-<junction x="109.22" y="132.08"/>
-</segment>
-</net>
 <net name="GND" class="0">
 <segment>
@@
 <pinref part="GND5" gate="1" pin="GND"/>
 <wire x1="180.34" y1="114.3" x2="180.34" y2="106.68" width="0.1524" layer="91"/>
+</segment>
+<segment>
+<pinref part="J2" gate="G$1" pin="GNDBREAK"/>
+<pinref part="GND39" gate="1" pin="GND"/>
+<wire x1="88.9" y1="129.54" x2="93.98" y2="129.54" width="0.1524" layer="91"/>
+<wire x1="93.98" y1="129.54" x2="93.98" y2="127" width="0.1524" layer="91"/>
+<pinref part="J2" gate="G$1" pin="GND"/>
+<wire x1="93.98" y1="127" x2="93.98" y2="106.68" width="0.1524" layer="91"/>
+<wire x1="88.9" y1="127" x2="93.98" y2="127" width="0.1524" layer="91"/>
+<junction x="93.98" y="127"/>
 </segment>
 </net>
@@
 <wire x1="180.34" y1="121.92" x2="180.34" y2="132.08" width="0.1524" layer="91"/>
 <junction x="180.34" y="132.08"/>
+</segment>
+</net>
+<net name="DEETE" class="0">
+<segment>
+<pinref part="U1" gate="G$1" pin="IN"/>
+<wire x1="129.54" y1="132.08" x2="121.92" y2="132.08" width="0.1524" layer="91"/>
+<pinref part="U1" gate="G$1" pin="EN"/>
+<wire x1="121.92" y1="132.08" x2="109.22" y2="132.08" width="0.1524" layer="91"/>
+<wire x1="129.54" y1="127" x2="121.92" y2="127" width="0.1524" layer="91"/>
+<wire x1="121.92" y1="127" x2="121.92" y2="132.08" width="0.1524" layer="91"/>
+<junction x="121.92" y="132.08"/>
+<pinref part="C1" gate="G$1" pin="+"/>
+<wire x1="109.22" y1="121.92" x2="109.22" y2="132.08" width="0.1524" layer="91"/>
+<pinref part="J2" gate="G$1" pin="PWR"/>
+<wire x1="88.9" y1="132.08" x2="109.22" y2="132.08" width="0.1524" layer="91"/>
+<junction x="109.22" y="132.08"/>
 </segment>
 </net>
@@
 </nets>
 </sheet>
+<sheet>
+<plain>
+<text x="5.08" y="167.64" size="5.08" layer="94">Clock</text>
+</plain>
+<instances>
+<instance part="FRAME5" gate="G$1" x="0" y="0"/>
+<instance part="DISP1" gate="G$1" x="60.96" y="91.44"/>
+</instances>
+<busses>
+</busses>
+<nets>
+</nets>
+</sheet>

Commit message: adicionado mais 2 CIs e mais LEDs, total 45
Parts:
- removed DISP1: YSD-439AR6B-35, SparkFun-LED:7-SEGMENT-4DIGIT-10MM-RED
- added D28, D29, D30, D31, D32, D33, D34, D35, D36, D37, D38, D39, D40, D41, D42, D43, D44, D45, D46: BLUE, SparkFun-LED:LED-BLUE0603
- added IC5, IC6, IC7: 74HC595D, 74xx-eu:74HC595D
- added LED1: YSD-439AR6B-35, SparkFun-LED:7-SEGMENT-4DIGIT-10MM-RED
- added Q1, Q2, Q3, Q4: 600mA/40V, SparkFun-DiscreteSemi:TRANS_NPN-MMBT2222AL
- added R29, R30, R31, R32, R33, R34, R35, R36, R37, R38, R39, R40, R41, R42, R43, R44, R45, R46, R47, R48, R49, R50, R51, R52, R53, R54, R55, R56, R57, R58: 510, SparkFun-Resistors:470OHM1/10W1%(0603)
- IC1: value 74HC595D -> 4511D; device 74xx-eu:74HC595D -> 45xx:4511D
- J1: value FEMALE 2x3 -> POWER_JACK; device SparkFun-Connectors:CONN_03X2FEMALE -> SparkFun-Connectors:POWER_JACK
- J2: value POWER_JACK -> FEMALE 2x3; device SparkFun-Connectors:POWER_JACK -> SparkFun-Connectors:CONN_03X2FEMALE
- R10, R11, R12, R13, R3, R4, R5, R6, R7, R8, R9: value 510 -> 470; device SparkFun-Resistors:470OHM1/10W1%(0603) -> SparkFun-Resistors:470OHM-0603-1/10W-1%
- renumbered LEDPWR to D1, S2 to S1
Connections:
- new net D28: IC7A.QC, R40.2
- new net D29: IC7A.QD, R41.2
- new net D30: IC7A.QE, R42.2
- new net D31: IC7A.QF, R43.2
- new net D32: IC7A.QG, R44.2
- new net D33: IC7A.QH, R45.2
- new net D34: IC2A.QA, R46.2
- new net D35: IC2A.QB, R47.2
- new net D36: IC2A.QC, R48.2
- new net D37: IC2A.QD, R49.2
- new net D38: IC2A.QE, R50.2
- new net D39: IC2A.QF, R51.2
- new net D40: IC2A.QG, R52.2
- new net D41: IC2A.QH, R53.2
- new net D42: IC3A.QA, R54.2
- new net D43: IC3A.QB, R55.2
- new net D44: IC3A.QC, R56.2
- new net D45: IC3A.QD, R57.2
- new net D46: IC3A.QE, R58.2
- new net D47: IC3A.QF
- new net N$104: IC5A.QH*, IC6A.SER
- new net N$31: IC1A.D, R9.1
- new net N$33: IC1A.C, R8.1
- new net N$34: IC1A.B, R7.1
- new net N$35: IC1A.A, R6.1
- new net N$36: IC1A.E, R10.1
- new net N$37: IC1A.F, R11.1
- new net N$38: IC1A.G, R12.1
- new net N$39: LED1.A, R6.2
- new net N$42: LED1.B, R7.2
- new net N$43: LED1.C, R8.2
- new net N$44: LED1.D, R9.2
- new net N$45: LED1.E, R10.2
- new net N$46: LED1.F, R11.2
- new net N$47: LED1.G, R12.2
- new net N$48: LED1.DIG4, Q4.E
- new net N$49: LED1.DIG3, Q3.E
- new net N$50: LED1.DIG2, Q2.E
- new net N$51: LED1.DIG1, Q1.E
- new net N$52: Q2.B, R4.2
- new net N$53: Q4.B, R13.2
- new net N$54: Q3.B, R5.2
- new net N$55: Q1.B, R3.2
- new net N$56: D28.A, R40.1
- new net N$57: D29.A, R41.1
- new net N$58: D30.A, R42.1
- new net N$59: D31.A, R43.1
- new net N$60: D32.A, R44.1
- new net N$61: D33.A, R45.1
- new net N$62: D34.A, R46.1
- new net N$64: D35.A, R47.1
- new net N$65: D36.A, R48.1
- new net N$66: D37.A, R49.1
- new net N$67: D38.A, R50.1
- new net N$68: D39.A, R51.1
- new net N$69: D40.A, R52.1
- new net N$70: D41.A, R53.1
- new net N$71: D42.A, R54.1
- new net N$72: D43.A, R55.1
- new net N$73: D44.A, R56.1
- new net N$74: D45.A, R57.1
- new net N$75: D46.A, R58.1
- new net OUT: IC2A.SER, IC7A.QH*
- net D10: now also IC5A.QA, R22.2; no longer IC2A.QA, R11.2
- net D11: now also IC5A.QB, R23.2; no longer IC2A.QB, R12.2
- net D12: now also IC5A.QC, R24.2; no longer IC2A.QC, R13.2
- net D13: now also IC5A.QD, R25.2; no longer IC2A.QD, R14.2
- net D14: now also IC5A.QE, R26.2; no longer IC2A.QE, R15.2
- net D15: now also IC5A.QF, R27.2; no longer IC2A.QF, R16.2
- net D16: now also IC5A.QG, R28.2; no longer IC2A.QG, R17.2
- net D17: now also IC5A.QH, R29.2; no longer IC2A.QH, R18.2
- net D18: now also IC6A.QA, R30.2; no longer IC3A.QA, R19.2
- net D19: now also IC6A.QB, R31.2; no longer IC3A.QB, R20.2
- net D2: now also IC4A.QA, R14.2; no longer IC1A.QA, R3.2
- net D20: now also IC6A.QC, R32.2; no longer IC3A.QC, R21.2
- net D21: now also IC6A.QD, R33.2; no longer IC3A.QD, R22.2
- net D22: now also IC6A.QE, R34.2; no longer IC3A.QE, R23.2
- net D23: now also IC6A.QF, R35.2; no longer IC3A.QF, R24.2
- net D24: now also IC6A.QG, R36.2; no longer IC3A.QG, R25.2
- net D25: now also IC6A.QH, R37.2; no longer IC3A.QH, R26.2
- net D26: now also IC7A.QA, R38.2; no longer IC4A.QA, R27.2
- net D27: now also IC7A.QB, R39.2; no longer IC4A.QB, R28.2
- net D3: now also IC4A.QB, R15.2; no longer IC1A.QB, R4.2
- net D4: now also IC4A.QC, R16.2; no longer IC1A.QC, R5.2
- net D5: now also IC4A.QD, R17.2; no longer IC1A.QD, R6.2
- net D6: now also IC4A.QE, R18.2; no longer IC1A.QE, R7.2
- net D7: now also IC4A.QF, R19.2; no longer IC1A.QF, R8.2
- net D8: now also IC4A.QG, R20.2; no longer IC1A.QG, R9.2
- net D9: now also IC4A.QH, R21.2; no longer IC1A.QH, R10.2
- net DEETE: now also J1.PWR; no longer J2.PWR
- net DTR: now also J2.6; no longer J1.6
- net GND: now also D28.C, D29.C, D30.C, D31.C, D32.C, D33.C, D34.C, D35.C, D36.C, D37.C, D38.C, D39.C, D40.C, D41.C, D42.C, D43.C, D44.C, D45.C, D46.C, IC5A.G, IC6A.G, IC7A.G, J1.GND, J1.GNDBREAK, J2.1; no longer IC1A.G, J1.1, J2.GND, J2.GNDBREAK
- net LED_RCK: now also IC5A.RCK, IC6A.RCK, IC7A.RCK; no longer IC1A.RCK
- net LED_SCK: now also IC5A.SCK, IC6A.SCK, IC7A.SCK; no longer IC1A.SCK
- net LED_SERIAL: now also IC4A.SER; no longer IC1A.SER
- net N$1: now also R14.1; no longer R3.1
- net N$10: now also R23.1; no longer R12.1
- net N$11: now also R24.1; no longer R13.1
- net N$12: now also R25.1; no longer R14.1
- net N$13: now also R26.1; no longer R15.1
- net N$14: now also R27.1; no longer R16.1
- net N$15: now also R28.1; no longer R17.1
- net N$16: now also R29.1; no longer R18.1
- net N$17: now also R30.1; no longer R19.1
- net N$18: now also R31.1; no longer R20.1
- net N$19: now also R32.1; no longer R21.1
- net N$2: now also R15.1; no longer R4.1
- net N$20: now also R33.1; no longer R22.1
- net N$21: now also R34.1; no longer R23.1
- net N$22: now also R35.1; no longer R24.1
- net N$23: now also R36.1; no longer R25.1
- net N$24: now also R37.1; no longer R26.1
- net N$25: now also R38.1; no longer R27.1
- net N$26: now also R39.1; no longer R28.1
- net N$3: now also R16.1; no longer R5.1
- net N$4: now also R17.1; no longer R6.1
- net N$40: now also IC4A.QH*, IC5A.SER; no longer IC1A.QH*, IC2A.SER
- net N$41: now also IC6A.QH*, IC7A.SER; no longer IC3A.QH*, IC4A.SER
- net N$5: now also R18.1; no longer R7.1
- net N$6: now also R19.1; no longer R8.1
- net N$7: now also R20.1; no longer R9.1
- net N$8: now also R21.1; no longer R10.1
- net N$9: now also R22.1; no longer R11.1
- net RX: now also J2.3; no longer J1.3
- net TX: now also J2.4; no longer J1.4
- net VCC: now also IC5A.SCL, IC6A.SCL, IC7A.SCL, J2.2; no longer IC1A.SCL, J1.2

Commit message: finalizada
Parts:
- J1: value POWER_JACK -> (none); device SparkFun-Connectors:POWER_JACK -> SparkFun-Connectors:CONN_02
Connections:
- removed net D47: IC3A.QF
- new net BCD_A: IC1A.IA, U2.PC0(ADC0)
- new net BCD_B: IC1A.IB, U2.PC1(ADC1)
- new net BCD_C: IC1A.IC, U2.PC2(ADC2)
- new net BCD_D: IC1A.ID, U2.PC3(ADC3)
- new net DISP_D1: R3.1, U2.PC4(ADC4/SDA)
- new net DISP_D2: R4.1, U2.PC5(ADC5/SCL)
- new net DISP_D3: R5.1, U2.ADC6
- new net DISP_D4: R13.1, U2.ADC7
- net DEETE: now also J1.2; no longer J1.PWR
- net GND: now also IC1A.LE, J1.1; no longer J1.GND, J1.GNDBREAK
- net VCC: now also IC1A.BI, IC1A.LT, Q1.C, Q2.C, Q3.C, Q4.C
Other:
- moved on the sheet: J1, Q2, Q3, Q4, R13, R4, R5
